File: superseded/kha-bgt-subrack/kha-bgt-main-reva/kicad/kha-bgt-main-front.kicad_pcb (KiCad board)
At the start: 2 copper layers, 40.6 x 128.5 mm, 0 parts

Commit message: .
Other:
- outline, holes or cut-outs redrawn
- board text added: "https://github.com/kiu/kha kha-bgt-main-front REV A"
- board text removed: "https://github.com/kiu/kha kha-bgt-main-front REV B"
